Commit message: Initial commit: Added mecanum bot simulation, SLAM, and waypoint follower

File: urdf/mecanum_bot.urdf.xacro (robot description, xacro)
@@ -28,11 +28,4 @@
              izz="${mass/2.0*r*r}"/>
   </xacro:macro>
-   <!-- ================= BASE LINK ================= -->
-  <link name="base_footprint"/>
-  <joint name="base_footprint_joint" type="fixed">
-    <parent link="base_footprint"/>
-    <child link="base_link"/>
-    <origin xyz="0 0 ${wheel_radius}" rpy="0 0 0"/>
-  </joint>
   <link name="base_link">
     <visual>
